Commit message: updated gazebo elements to support multiples/renaming
-added ${name} param to mimic joint names to match corresponding urdf
-moved control plugin to bh_alone.urdf.xacro so multiple hands can be included into other robots without a name collision in gazebo

File: barrett_hand_description/robots/bh_alone.urdf.xacro (robot description, xacro)
@@ -27,3 +27,10 @@
 		<origin xyz="0 0 0" rpy="0 0 0" />
 	</xacro:bhand_macro>
+	<gazebo>
+	    <plugin name="ros_control" filename="libgazebo_ros_control.so">
+	       <robotNamespace>/</robotNamespace>
+	       <controlPeriod>0.001</controlPeriod>
+	       <robotSimType>gazebo_ros_control/DefaultRobotHWSim</robotSimType>
+	    </plugin>
+    </gazebo>
 </robot>

File: barrett_hand_description/urdf/bh282.gazebo.xacro (robot description, xacro)
@@ -2,16 +2,8 @@
 <robot xmlns:xacro="http://ros.org/wiki/xacro">
   <xacro:macro name="bh_gazebo" params="name">
-	<!-- ros_control plugin -->
-	<gazebo>
-		<plugin name="ros_control" filename="libgazebo_ros_control.so">
-		   <robotNamespace>/</robotNamespace>
-		   <controlPeriod>0.001</controlPeriod>
-		   <robotSimType>gazebo_ros_control/DefaultRobotHWSim</robotSimType>
-		</plugin>
-	</gazebo>
 	<gazebo>
 	   	<plugin name="mimic_plugin" filename="libgazebo_mimic_plugin.so">
-       		   <joint>bh_j11_joint</joint>
-       		   <mimicJoint>bh_j21_joint</mimicJoint>
+       		   <joint>${name}_j11_joint</joint>
+       		   <mimicJoint>${name}_j21_joint</mimicJoint>
        		   <multiplier>1</multiplier>
        		</plugin>
@@ -19,6 +11,6 @@
 	<gazebo>
 	    	<plugin name="mimic_plugin" filename="libgazebo_mimic_plugin.so">
-       		   <joint>bh_j12_joint</joint>
-       		   <mimicJoint>bh_j13_joint</mimicJoint>
+       		   <joint>${name}_j12_joint</joint>
+       		   <mimicJoint>${name}_j13_joint</mimicJoint>
        		   <multiplier>0.344</multiplier>
        		</plugin>
@@ -26,6 +18,6 @@
 	<gazebo>
 	    	<plugin name="mimic_plugin" filename="libgazebo_mimic_plugin.so">
-       		   <joint>bh_j22_joint</joint>
-       		   <mimicJoint>bh_j23_joint</mimicJoint>
+       		   <joint>${name}_j22_joint</joint>
+       		   <mimicJoint>${name}_j23_joint</mimicJoint>
        		   <multiplier>0.344</multiplier>
        		</plugin>
@@ -33,6 +25,6 @@
 	<gazebo>
 	    	<plugin name="mimic_plugin" filename="libgazebo_mimic_plugin.so">
-       		   <joint>bh_j32_joint</joint>
-       		   <mimicJoint>bh_j33_joint</mimicJoint>
+       		   <joint>${name}_j32_joint</joint>
+       		   <mimicJoint>${name}_j33_joint</mimicJoint>
        		   <multiplier>0.344</multiplier>
        		</plugin>
