Commit message: change bh280 to mimic joints

File: barrett_hand_description/urdf/bh280.urdf.xacro (robot description, xacro)
@@ -114,4 +114,5 @@
 			<limit effort="${joint_effort_limit}" lower="0.0" upper="0.84" velocity="${joint_velocity_limit}"/>
 			<dynamics damping="${joint_damping}" friction="${joint_friction}"/>
+			<mimic joint="${name}_j32_joint" multiplier="0.344" />
 		</joint>
 		<transmission name="${name}_j33_transmission">
@@ -241,4 +242,5 @@
 			<limit effort="${joint_effort_limit}" lower="0.0" upper="0.84" velocity="${joint_velocity_limit}"/>
 			<dynamics damping="${joint_damping}" friction="${joint_friction}"/>
+			<mimic joint="${name}_j12_joint" multiplier="0.344" />
 		</joint>
 		<transmission name="${name}_j13_transmission">
@@ -283,4 +285,5 @@
 			<limit effort="${joint_effort_limit}" lower="0" upper="3.1416" velocity="${joint_velocity_limit}"/>
 			<dynamics damping="${joint_damping}" friction="${joint_friction}"/>
+			<mimic joint="${name}_j11_joint" multiplier="1" />
 		</joint>
 		<transmission name="${name}_j21_transmission">
@@ -368,4 +371,5 @@
 			<limit effort="${joint_effort_limit}" lower="0.0" upper="0.84" velocity="${joint_velocity_limit}"/>
 			<dynamics damping="${joint_damping}" friction="${joint_friction}"/>
+			<mimic joint="${name}_j22_joint" multiplier="0.344" />
 		</joint>
 		<transmission name="${name}_j23_transmission">

File: barrett_hand_description/urdf/bh282.gazebo.xacro (robot description, xacro)
@@ -2,4 +2,5 @@
 <robot xmlns:xacro="http://ros.org/wiki/xacro">
   <xacro:macro name="bh_gazebo" params="name">
+<!--
 	<gazebo>
 	   	<plugin name="mimic_plugin" filename="libgazebo_mimic_plugin.so">
@@ -30,4 +31,5 @@
        		</plugin>
         </gazebo>
+-->
 	<gazebo reference="${name}_base_link">
 		<material>Gazebo/White</material>

Commit message: cleaned up bh280 mimic joints

File: barrett_hand_description/urdf/bh280.urdf.xacro (robot description, xacro)
@@ -112,7 +112,7 @@
 			<origin xyz="-0.069936 0.003 0" rpy="0 0 0" />
 			<axis xyz="0 0 -1"/>
+			<mimic joint="${name}_j32_joint" multiplier="${0.84/2.44}" />
 			<limit effort="${joint_effort_limit}" lower="0.0" upper="0.84" velocity="${joint_velocity_limit}"/>
 			<dynamics damping="${joint_damping}" friction="${joint_friction}"/>
-			<mimic joint="${name}_j32_joint" multiplier="0.344" />
 		</joint>
 		<transmission name="${name}_j33_transmission">
@@ -240,7 +240,7 @@
 			<origin xyz="-0.069936 0.003 0" rpy="0 0 0" />
 			<axis xyz="0 0 -1"/>
+			<mimic joint="${name}_j12_joint" multiplier="${0.84/2.44}" />
 			<limit effort="${joint_effort_limit}" lower="0.0" upper="0.84" velocity="${joint_velocity_limit}"/>
 			<dynamics damping="${joint_damping}" friction="${joint_friction}"/>
-			<mimic joint="${name}_j12_joint" multiplier="0.344" />
 		</joint>
 		<transmission name="${name}_j13_transmission">
@@ -283,7 +283,7 @@
 			<origin xyz="-0.025 0 0.0415" rpy="0 0 -1.5708" />
 			<axis xyz="0 0 1"/>
+			<mimic joint="${name}_j11_joint" multiplier="1" />
 			<limit effort="${joint_effort_limit}" lower="0" upper="3.1416" velocity="${joint_velocity_limit}"/>
 			<dynamics damping="${joint_damping}" friction="${joint_friction}"/>
-			<mimic joint="${name}_j11_joint" multiplier="1" />
 		</joint>
 		<transmission name="${name}_j21_transmission">
@@ -369,7 +369,7 @@
 			<origin xyz="-0.069936 0.003 0" rpy="0 0 0" />
 			<axis xyz="0 0 -1"/>
+			<mimic joint="${name}_j22_joint" multiplier="${0.84/2.44}" />
 			<limit effort="${joint_effort_limit}" lower="0.0" upper="0.84" velocity="${joint_velocity_limit}"/>
 			<dynamics damping="${joint_damping}" friction="${joint_friction}"/>
-			<mimic joint="${name}_j22_joint" multiplier="0.344" />
 		</joint>
 		<transmission name="${name}_j23_transmission">

File: barrett_hand_description/urdf/bh282.gazebo.xacro (robot description, xacro)
@@ -2,5 +2,4 @@
 <robot xmlns:xacro="http://ros.org/wiki/xacro">
   <xacro:macro name="bh_gazebo" params="name">
-<!--
 	<gazebo>
 	   	<plugin name="mimic_plugin" filename="libgazebo_mimic_plugin.so">
@@ -31,5 +30,4 @@
        		</plugin>
         </gazebo>
--->
 	<gazebo reference="${name}_base_link">
 		<material>Gazebo/White</material>

Commit message: Added tactile info

File: barrett_hand_description/urdf/bh280.urdf.xacro (robot description, xacro)
@@ -3,4 +3,5 @@
 	<!-- Import all Gazebo-customization elements, including Gazebo colors -->
 	<xacro:include filename="$(find barrett_hand_description)/urdf/bh282.gazebo.xacro" />
+	<xacro:include filename="$(find barrett_hand_description)/urdf/bh280_tactile.urdf.xacro" />
 	<!-- Constants for robot dimensions -->
 	<xacro:property name="PI" value="3.1415926535897931"/>
@@ -384,5 +385,26 @@
 			</actuator>
 		</transmission>
-		<xacro:bh_gazebo name="${name}"/>
+		<!-- Imaginary joints for transform from tactile sensors -->
+		<!-- Radian value obtained from graspit description of 40 degrees -->
+		<joint name="${name}_finger_14_joint" type="fixed">
+			<parent link="${name}_finger_13_link"/>
+			<child link="${name}_finger_14_link"/>
+			<origin xyz="0 0 0" rpy="0 0 0.698132" />
+		</joint>
+		<link name="${name}_finger_14_link"/>
+		<joint name="${name}_finger_24_joint" type="fixed">
+			<parent link="${name}_finger_23_link"/>
+			<child link="${name}_finger_24_link"/>
+			<origin xyz="0 0 0" rpy="0 0 0.698132" />
+		</joint>
+		<link name="${name}_finger_24_link"/>
+		<joint name="${name}_finger_34_joint" type="fixed">
+			<parent link="${name}_finger_33_link"/>
+			<child link="${name}_finger_34_link"/>
+			<origin xyz="0 0 0" rpy="0 0 0.698132" />
+		</joint>
+		<link name="${name}_finger_34_link"/>
+		<!-- Auto generated tactile sensor links -->
+		<xacro:bh_tactile name="bh"/>
 	</xacro:macro>
 </robot>
